File: macro_keyboard_pcb/macro_keyboard_pcb.sch (KiCad schematic (older format))
At the start: 56 parts

Commit message: Add LED circuit, assign footprints
Parts:
- added C1, C2: C_Small, Capacitor_SMD:C_0603_1608Metric_Pad1.08x0.95mm_HandSolder, symbol Device:C_Small
- added D26: WS2812B, LED_SMD:LED_WS2812B_PLCC4_5.0x5.0mm_P3.2mm, symbol LED:WS2812B
- added R1: 360, Resistor_SMD:R_0603_1608Metric_Pad0.98x0.95mm_HandSolder, symbol Device:R_Small
- RV1, RV2, RV3, RV4, RV5: renamed from RV?; footprint (none) -> Potentiometer_THT:Potentiometer_ACP_CA9-V10_Vertical
- SW1, SW10, SW11, SW12, SW13, SW14, SW15, SW16, SW17, SW18, SW19, SW2, SW20, SW21, SW22, SW23, SW24, SW25, SW3, SW4, SW5, SW6, SW7, SW8, SW9: renamed from SW?; footprint (none) -> CherryMX:CherryMX_1.00u
- U1: renamed from U?; footprint (none) -> promicro:ProMicro
- gave numbers to parts that had none: 25
Connections:
- net +5V: now also RV1.3, RV2.3, RV3.3, RV4.3, RV5.3, C1.1, C2.1, D26.1 (VDD)
- net COL0: now also U1.8 (C6)
- net COL1: now also U1.9 (D7)
- net COL2: now also U1.10 (E6)
- net COL3: now also U1.11 (B4)
- net COL4: now also U1.12 (B5)
- net GND: now also RV1.1, RV2.1, RV3.1, RV4.1, RV5.1, C1.2, C2.2, D26.3 (VSS)
- net ROW0: now also U1.2 (RX)
- net ROW1: now also U1.1 (TX)
- net ROW2: now also U1.5 (SCL)
- net ROW3: now also U1.6 (SDA)
- net ROW4: now also U1.7 (D4)
- net POT4: now reaches U1.13 (B6)
- net POT4: now also RV5.2
- net LED_DATA: now reaches U1.14 (B2)
- net LED_DATA: now also R1.1
- net POT0: now reaches U1.17 (F7)
- net POT0: now also RV1.2
- net POT1: now reaches U1.18 (F6)
- net POT1: now also RV2.2
- net POT2: now reaches U1.19 (F5)
- net POT2: now also RV3.2
- net POT3: now reaches U1.20 (F4)
- net POT3: now also RV4.2
- new net: D26.4 (DIN), R1.2
Other:
- moved on the sheet: RV1, RV2, RV3, RV4, RV5

Commit message: WIP adding routes
Parts:
- D1, D10, D11, D12, D13, D14, D15, D16, D17, D18, D19, D2, D20, D21, D22, D23, D24, D25, D3, D4, D5, D6, D7, D8, D9: footprint Diode_THT:D_DO-35_SOD27_P7.62mm_Horizontal -> Diode_SMD:D_SOD-123
Connections:
- net COL2: now also SW11.1
- net at D12.2 (A): now also SW12.2
- net at D11.2 (A): now also SW11.2; no longer SW12.2
Other:
- moved on the sheet: SW11, SW12
Changed lines of the file:
@@
 F 0 "D2" V 1996 3120 50  0000 R CNN
 F 1 "1N4148" V 1905 3120 50  0000 R CNN
-F 2 "Diode_THT:D_DO-35_SOD27_P7.62mm_Horizontal" H 1950 3025 50  0001 C CNN
+F 2 "Diode_SMD:D_SOD-123" H 1950 3025 50  0001 C CNN
 F 3 "https://assets.nexperia.com/documents/data-sheet/1N4148_1N4448.pdf" H 1950 3200 50  0001 C CNN
 	1    1950 3200
@@
 F 0 "D7" V 2996 3120 50  0000 R CNN
 F 1 "1N4148" V 2905 3120 50  0000 R CNN
-F 2 "Diode_THT:D_DO-35_SOD27_P7.62mm_Horizontal" H 2950 3025 50  0001 C CNN
+F 2 "Diode_SMD:D_SOD-123" H 2950 3025 50  0001 C CNN
 F 3 "https://assets.nexperia.com/documents/data-sheet/1N4148_1N4448.pdf" H 2950 3200 50  0001 C CNN
 	1    2950 3200
@@
 F 0 "D12" V 3996 3120 50  0000 R CNN
 F 1 "1N4148" V 3905 3120 50  0000 R CNN
-F 2 "Diode_THT:D_DO-35_SOD27_P7.62mm_Horizontal" H 3950 3025 50  0001 C CNN
+F 2 "Diode_SMD:D_SOD-123" H 3950 3025 50  0001 C CNN
 F 3 "https://assets.nexperia.com/documents/data-sheet/1N4148_1N4448.pdf" H 3950 3200 50  0001 C CNN
 	1    3950 3200
@@
 F 0 "D17" V 4996 3120 50  0000 R CNN
 F 1 "1N4148" V 4905 3120 50  0000 R CNN
-F 2 "Diode_THT:D_DO-35_SOD27_P7.62mm_Horizontal" H 4950 3025 50  0001 C CNN
+F 2 "Diode_SMD:D_SOD-123" H 4950 3025 50  0001 C CNN
 F 3 "https://assets.nexperia.com/documents/data-sheet/1N4148_1N4448.pdf" H 4950 3200 50  0001 C CNN
 	1    4950 3200
@@
 F 0 "D22" V 5996 3120 50  0000 R CNN
 F 1 "1N4148" V 5905 3120 50  0000 R CNN
-F 2 "Diode_THT:D_DO-35_SOD27_P7.62mm_Horizontal" H 5950 3025 50  0001 C CNN
+F 2 "Diode_SMD:D_SOD-123" H 5950 3025 50  0001 C CNN
 F 3 "https://assets.nexperia.com/documents/data-sheet/1N4148_1N4448.pdf" H 5950 3200 50  0001 C CNN
 	1    5950 3200
@@
 F 0 "D23" V 5996 4120 50  0000 R CNN
 F 1 "1N4148" V 5905 4120 50  0000 R CNN
-F 2 "Diode_THT:D_DO-35_SOD27_P7.62mm_Horizontal" H 5950 4025 50  0001 C CNN
+F 2 "Diode_SMD:D_SOD-123" H 5950 4025 50  0001 C CNN
 F 3 "https://assets.nexperia.com/documents/data-sheet/1N4148_1N4448.pdf" H 5950 4200 50  0001 C CNN
 	1    5950 4200
@@
 F 0 "D18" V 4996 4120 50  0000 R CNN
 F 1 "1N4148" V 4905 4120 50  0000 R CNN
-F 2 "Diode_THT:D_DO-35_SOD27_P7.62mm_Horizontal" H 4950 4025 50  0001 C CNN
+F 2 "Diode_SMD:D_SOD-123" H 4950 4025 50  0001 C CNN
 F 3 "https://assets.nexperia.com/documents/data-sheet/1N4148_1N4448.pdf" H 4950 4200 50  0001 C CNN
 	1    4950 4200
@@
 F 0 "D13" V 3996 4120 50  0000 R CNN
 F 1 "1N4148" V 3905 4120 50  0000 R CNN
-F 2 "Diode_THT:D_DO-35_SOD27_P7.62mm_Horizontal" H 3950 4025 50  0001 C CNN
+F 2 "Diode_SMD:D_SOD-123" H 3950 4025 50  0001 C CNN
 F 3 "https://assets.nexperia.com/documents/data-sheet/1N4148_1N4448.pdf" H 3950 4200 50  0001 C CNN
 	1    3950 4200
@@
 F 0 "D8" V 2996 4120 50  0000 R CNN
 F 1 "1N4148" V 2905 4120 50  0000 R CNN
-F 2 "Diode_THT:D_DO-35_SOD27_P7.62mm_Horizontal" H 2950 4025 50  0001 C CNN
+F 2 "Diode_SMD:D_SOD-123" H 2950 4025 50  0001 C CNN
 F 3 "https://assets.nexperia.com/documents/data-sheet/1N4148_1N4448.pdf" H 2950 4200 50  0001 C CNN
 	1    2950 4200
@@
 F 0 "D3" V 1996 4120 50  0000 R CNN
 F 1 "1N4148" V 1905 4120 50  0000 R CNN
-F 2 "Diode_THT:D_DO-35_SOD27_P7.62mm_Horizontal" H 1950 4025 50  0001 C CNN
+F 2 "Diode_SMD:D_SOD-123" H 1950 4025 50  0001 C CNN
 F 3 "https://assets.nexperia.com/documents/data-sheet/1N4148_1N4448.pdf" H 1950 4200 50  0001 C CNN
 	1    1950 4200
@@
 F 0 "D4" V 1996 5120 50  0000 R CNN
 F 1 "1N4148" V 1905 5120 50  0000 R CNN
-F 2 "Diode_THT:D_DO-35_SOD27_P7.62mm_Horizontal" H 1950 5025 50  0001 C CNN
+F 2 "Diode_SMD:D_SOD-123" H 1950 5025 50  0001 C CNN
 F 3 "https://assets.nexperia.com/documents/data-sheet/1N4148_1N4448.pdf" H 1950 5200 50  0001 C CNN
 	1    1950 5200
@@
 F 0 "D9" V 2996 5120 50  0000 R CNN
 F 1 "1N4148" V 2905 5120 50  0000 R CNN
-F 2 "Diode_THT:D_DO-35_SOD27_P7.62mm_Horizontal" H 2950 5025 50  0001 C CNN
+F 2 "Diode_SMD:D_SOD-123" H 2950 5025 50  0001 C CNN
 F 3 "https://assets.nexperia.com/documents/data-sheet/1N4148_1N4448.pdf" H 2950 5200 50  0001 C CNN
 	1    2950 5200
@@
 F 0 "D14" V 3996 5120 50  0000 R CNN
 F 1 "1N4148" V 3905 5120 50  0000 R CNN
-F 2 "Diode_THT:D_DO-35_SOD27_P7.62mm_Horizontal" H 3950 5025 50  0001 C CNN
+F 2 "Diode_SMD:D_SOD-123" H 3950 5025 50  0001 C CNN
 F 3 "https://assets.nexperia.com/documents/data-sheet/1N4148_1N4448.pdf" H 3950 5200 50  0001 C CNN
 	1    3950 5200
@@
 F 0 "D19" V 4996 5120 50  0000 R CNN
 F 1 "1N4148" V 4905 5120 50  0000 R CNN
-F 2 "Diode_THT:D_DO-35_SOD27_P7.62mm_Horizontal" H 4950 5025 50  0001 C CNN
+F 2 "Diode_SMD:D_SOD-123" H 4950 5025 50  0001 C CNN
 F 3 "https://assets.nexperia.com/documents/data-sheet/1N4148_1N4448.pdf" H 4950 5200 50  0001 C CNN
 	1    4950 5200
@@
 F 0 "D24" V 5996 5120 50  0000 R CNN
 F 1 "1N4148" V 5905 5120 50  0000 R CNN
-F 2 "Diode_THT:D_DO-35_SOD27_P7.62mm_Horizontal" H 5950 5025 50  0001 C CNN
+F 2 "Diode_SMD:D_SOD-123" H 5950 5025 50  0001 C CNN
 F 3 "https://assets.nexperia.com/documents/data-sheet/1N4148_1N4448.pdf" H 5950 5200 50  0001 C CNN
 	1    5950 5200
@@
 F 0 "D25" V 5996 6120 50  0000 R CNN
 F 1 "1N4148" V 5905 6120 50  0000 R CNN
-F 2 "Diode_THT:D_DO-35_SOD27_P7.62mm_Horizontal" H 5950 6025 50  0001 C CNN
+F 2 "Diode_SMD:D_SOD-123" H 5950 6025 50  0001 C CNN
 F 3 "https://assets.nexperia.com/documents/data-sheet/1N4148_1N4448.pdf" H 5950 6200 50  0001 C CNN
 	1    5950 6200
@@
 F 0 "D20" V 4996 6120 50  0000 R CNN
 F 1 "1N4148" V 4905 6120 50  0000 R CNN
-F 2 "Diode_THT:D_DO-35_SOD27_P7.62mm_Horizontal" H 4950 6025 50  0001 C CNN
+F 2 "Diode_SMD:D_SOD-123" H 4950 6025 50  0001 C CNN
 F 3 "https://assets.nexperia.com/documents/data-sheet/1N4148_1N4448.pdf" H 4950 6200 50  0001 C CNN
 	1    4950 6200
@@
 F 0 "D15" V 3996 6120 50  0000 R CNN
 F 1 "1N4148" V 3905 6120 50  0000 R CNN
-F 2 "Diode_THT:D_DO-35_SOD27_P7.62mm_Horizontal" H 3950 6025 50  0001 C CNN
+F 2 "Diode_SMD:D_SOD-123" H 3950 6025 50  0001 C CNN
 F 3 "https://assets.nexperia.com/documents/data-sheet/1N4148_1N4448.pdf" H 3950 6200 50  0001 C CNN
 	1    3950 6200
@@
 F 0 "D10" V 2996 6120 50  0000 R CNN
 F 1 "1N4148" V 2905 6120 50  0000 R CNN
-F 2 "Diode_THT:D_DO-35_SOD27_P7.62mm_Horizontal" H 2950 6025 50  0001 C CNN
+F 2 "Diode_SMD:D_SOD-123" H 2950 6025 50  0001 C CNN
 F 3 "https://assets.nexperia.com/documents/data-sheet/1N4148_1N4448.pdf" H 2950 6200 50  0001 C CNN
 	1    2950 6200
@@
 F 0 "D5" V 1996 6120 50  0000 R CNN
 F 1 "1N4148" V 1905 6120 50  0000 R CNN
-F 2 "Diode_THT:D_DO-35_SOD27_P7.62mm_Horizontal" H 1950 6025 50  0001 C CNN
+F 2 "Diode_SMD:D_SOD-123" H 1950 6025 50  0001 C CNN
 F 3 "https://assets.nexperia.com/documents/data-sheet/1N4148_1N4448.pdf" H 1950 6200 50  0001 C CNN
 	1    1950 6200
@@
 F 0 "D1" V 1996 2120 50  0000 R CNN
 F 1 "1N4148" V 1905 2120 50  0000 R CNN
-F 2 "Diode_THT:D_DO-35_SOD27_P7.62mm_Horizontal" H 1950 2025 50  0001 C CNN
+F 2 "Diode_SMD:D_SOD-123" H 1950 2025 50  0001 C CNN
 F 3 "https://assets.nexperia.com/documents/data-sheet/1N4148_1N4448.pdf" H 1950 2200 50  0001 C CNN
 	1    1950 2200
@@
 F 0 "D6" V 2996 2120 50  0000 R CNN
 F 1 "1N4148" V 2905 2120 50  0000 R CNN
-F 2 "Diode_THT:D_DO-35_SOD27_P7.62mm_Horizontal" H 2950 2025 50  0001 C CNN
+F 2 "Diode_SMD:D_SOD-123" H 2950 2025 50  0001 C CNN
 F 3 "https://assets.nexperia.com/documents/data-sheet/1N4148_1N4448.pdf" H 2950 2200 50  0001 C CNN
 	1    2950 2200
@@
 F 0 "D11" V 3996 2120 50  0000 R CNN
 F 1 "1N4148" V 3905 2120 50  0000 R CNN
-F 2 "Diode_THT:D_DO-35_SOD27_P7.62mm_Horizontal" H 3950 2025 50  0001 C CNN
+F 2 "Diode_SMD:D_SOD-123" H 3950 2025 50  0001 C CNN
 F 3 "https://assets.nexperia.com/documents/data-sheet/1N4148_1N4448.pdf" H 3950 2200 50  0001 C CNN
 	1    3950 2200
@@
 F 0 "D16" V 4996 2120 50  0000 R CNN
 F 1 "1N4148" V 4905 2120 50  0000 R CNN
-F 2 "Diode_THT:D_DO-35_SOD27_P7.62mm_Horizontal" H 4950 2025 50  0001 C CNN
+F 2 "Diode_SMD:D_SOD-123" H 4950 2025 50  0001 C CNN
 F 3 "https://assets.nexperia.com/documents/data-sheet/1N4148_1N4448.pdf" H 4950 2200 50  0001 C CNN
 	1    4950 2200
@@
 F 0 "D21" V 5996 2120 50  0000 R CNN
 F 1 "1N4148" V 5905 2120 50  0000 R CNN
-F 2 "Diode_THT:D_DO-35_SOD27_P7.62mm_Horizontal" H 5950 2025 50  0001 C CNN
+F 2 "Diode_SMD:D_SOD-123" H 5950 2025 50  0001 C CNN
 F 3 "https://assets.nexperia.com/documents/data-sheet/1N4148_1N4448.pdf" H 5950 2200 50  0001 C CNN
 	1    5950 2200
@@
 $EndComp
 $Comp
-L CherryMX:CherryMX SW12
-U 1 1 5FCC8EBB
-P 3750 2050
-F 0 "SW12" H 3750 2335 50  0000 C CNN
-F 1 "CherryMX" H 3750 2244 50  0000 C CNN
-F 2 "CherryMX:CherryMX_1.00u" H 3750 2075 50  0001 C CNN
-F 3 "" H 3750 2075 50  0001 C CNN
-	1    3750 2050
-	1    0    0    -1
-$EndComp
-$Comp
 L CherryMX:CherryMX SW16
 U 1 1 5FCC98A5
@@
 L CherryMX:CherryMX SW11
 U 1 1 5FCCD6A4
-P 3700 3050
-F 0 "SW11" H 3700 3335 50  0000 C CNN
-F 1 "CherryMX" H 3700 3244 50  0000 C CNN
-F 2 "CherryMX:CherryMX_1.00u" H 3700 3075 50  0001 C CNN
-F 3 "" H 3700 3075 50  0001 C CNN
-	1    3700 3050
+P 3750 2050
+F 0 "SW11" H 3750 2335 50  0000 C CNN
+F 1 "CherryMX" H 3750 2244 50  0000 C CNN
+F 2 "CherryMX:CherryMX_1.00u" H 3750 2075 50  0001 C CNN
+F 3 "" H 3750 2075 50  0001 C CNN
+	1    3750 2050
 	1    0    0    -1
 $EndComp
@@
 Connection ~ 3550 4050
 Wire Wire Line
-	3550 4050 3550 2050
+	3550 4050 3550 3050
 Connection ~ 3550 5050
 Wire Wire Line
@@
 Wire Wire Line
 	9650 4900 9400 4900
+Connection ~ 3550 3050
+Wire Wire Line
+	3550 3050 3550 2050
+$Comp
+L CherryMX:CherryMX SW12
+U 1 1 5FCC8EBB
+P 3750 3050
+F 0 "SW12" H 3750 3335 50  0000 C CNN
+F 1 "CherryMX" H 3750 3244 50  0000 C CNN
+F 2 "CherryMX:CherryMX_1.00u" H 3750 3075 50  0001 C CNN
+F 3 "" H 3750 3075 50  0001 C CNN
+	1    3750 3050
+	1    0    0    -1
+$EndComp
 $EndSCHEMATC
